File: transceiver_data_conversion.kicad_sch (KiCad schematic)
At the start: 10 parts, among them U3 MAX485E

Commit message: meeting today, need to rewire
Connections:
- net 5V: now also C10.1, C11.1
Changed lines of the file:
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@@
+	)
+	(junction
+		(at 95.25 97.79)
+		(diameter 0)
+		(color 0 0 0 0)
 	)
 	(junction
@@
 	(wire
 		(pts
+			(xy 106.68 97.79) (xy 106.68 100.33)
+		)
+		(stroke
+			(width 0)
+			(type default)
+		)
+	)
+	(wire
+		(pts
 			(xy 74.93 83.82) (xy 76.2 83.82)
 		)
@@
 	(wire
 		(pts
+			(xy 95.25 97.79) (xy 95.25 100.33)
+		)
+		(stroke
+			(width 0)
+			(type default)
+		)
+	)
+	(wire
+		(pts
 			(xy 144.78 72.39) (xy 144.78 77.47)
 		)
@@
 	(wire
 		(pts
-			(xy 95.25 100.33) (xy 106.68 100.33)
+			(xy 95.25 97.79) (xy 106.68 97.79)
 		)
 		(stroke
@@
 		(pts
 			(xy 151.13 82.55) (xy 151.13 97.79)
+		)
+		(stroke
+			(width 0)
+			(type default)
+		)
+	)
+	(wire
+		(pts
+			(xy 95.25 95.25) (xy 95.25 97.79)
 		)
 		(stroke
@@
 			(effects
 				(font
+					(size 1.27 1.27)
+				)
+				(justify left)
+				(hide yes)
+			)
+		)
+	)
+	(global_label "5V"
+		(shape output)
+		(at 95.25 95.25 0)
+		(fields_autoplaced yes)
+		(effects
+			(font
+				(size 1.27 1.27)
+			)
+			(justify left)
+		)
+		(property "Intersheetrefs" "${INTERSHEET_REFS}"
+			(at 100.5333 95.25 0)
+			(effects
+				(font
