File: X17-Data-Conversion.kicad_pcb (KiCad board)
At the start: 2 copper layers, 41.5 x 37.3 mm, 35 parts, among them J1 Conn_01x05, J4 Conn_01x12_Pin, SW1 1825910-6, U2 STM32F091CCTx, U3 MAX485E, U4 MAX7375AXR805+T, U5 AZ1117IH-3.3TRG1

Commit message: prep to start final (hopefully) layout
Parts:
- removed the C1 at (161.8, 99.3)
- removed C2, C3: 18pF, Capacitor_SMD:C_0603_1608Metric_Pad1.08x0.95mm_HandSolder
- removed R1: 10k, Resistor_SMD:R_0603_1608Metric_Pad0.98x0.95mm_HandSolder
- removed the R2 at (146.0, 70.5)
- removed R3: 4.7k, Resistor_SMD:R_0603_1608Metric_Pad0.98x0.95mm_HandSolder
- removed SW1: 1825910-6, footprints1:SW4_1825910-B_TEC
- moved R11 88.4 mm to (88.6, 107.8), turned to 0 degrees
- moved R9 86.4 mm to (88.6, 102.8)
- moved R10 83.0 mm to (88.6, 105.3)
- moved R8 82.3 mm to (88.6, 100.2)
- moved R7 77.9 mm to (88.6, 97.7)
- moved R6 77.7 mm to (88.6, 95.2)
- moved U3 77.0 mm to (95.0, 89.8)
- moved R4 73.6 mm to (103.4, 107.8), turned to 0 degrees
- moved C8 73.6 mm to (103.4, 97.7), turned to 0 degrees
- moved R5 73.1 mm to (88.6, 92.7)
- moved C9 73.1 mm to (103.4, 100.2), turned to 0 degrees
- moved J1 72.2 mm to (107.9, 88.8)
- moved C7 65.4 mm to (103.4, 95.2), turned to 0 degrees
- moved C4 65.0 mm to (103.4, 87.7)
- moved C6 63.9 mm to (103.4, 92.7), turned to 0 degrees
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Routing:
- net GND: track 120.5 -> 0.00 mm, vias 24 -> 0
- net NRST_PSB: track 78.4 -> 0.00 mm, vias 3 -> 0
- net 3.3V: track 61.1 -> 0.00 mm, vias 12 -> 0
- net 5V: track 49.9 -> 0.00 mm
- net I2C1_SCL: track 40.7 -> 0.00 mm, vias 1 -> 0
- net SWCLK: track 40.5 -> 0.00 mm
- net SWDIO: track 38.2 -> 0.00 mm, vias 1 -> 0
- net Net-(U2-PB1): track 24.7 -> 0.00 mm, vias 2 -> 0
- net Net-(U2-PB0): track 24.7 -> 0.00 mm
- net /OSC_IN: track 21.9 -> 0.00 mm
- net unconnected-(U2-PB3-Pad39): track 18.4 -> 0.00 mm, vias 2 -> 0
- net /OSC_OUT: track 17.3 -> 0.00 mm
- net A-: track 16.9 -> 0.00 mm
- net ALERT1: track 16.3 -> 0.00 mm
- net USART1_DE: track 13.7 -> 0.00 mm
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- removed copper zone on B.Cu, net 3.3V
- removed copper zone on F.Cu, net 5V
- removed copper zone on F.Cu, net GND
Other:
- board size 41.5 x 37.3 mm -> 41.5 x 30.7 mm

Commit message: hny!
lookinggood, happy new year!
Parts:
- moved R10 92.9 mm to (180.7, 92.9)
- moved R9 92.5 mm to (180.7, 94.4), turned to 180 degrees
- moved R11 90.9 mm to (178.4, 93.7), turned to -90 degrees
- moved R8 80.3 mm to (168.8, 96.1)
- moved R5 80.2 mm to (168.8, 91.6)
- moved R7 80.2 mm to (168.7, 94.7)
- moved R6 80.2 mm to (168.8, 93.2)
- moved C10 80.2 mm to (168.8, 87.3)
- moved C11 80.2 mm to (168.8, 88.9)
- moved U3 79.3 mm to (174.2, 93.7)
- moved R4 73.7 mm to (164.8, 67.0)
- moved D1 68.7 mm to (168.3, 67.1), turned to 180 degrees
- moved U2 49.1 mm to (161.6, 74.2)
- moved C13 44.5 mm to (144.3, 87.7), turned to 180 degrees
- moved C12 42.7 mm to (144.2, 90.1)
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Connections:
- J4 pad 2: DATA -> I2C1_SDA
- J4 pad 9: CLK -> I2C1_SCL
Routing:
- net 3.3V: track 0.00 -> 10.0 mm
- net 5V: track 0.00 -> 5.57 mm, vias 0 -> 1
- net GND: track 0.00 -> 5.40 mm, vias 0 -> 1
- net USART1_DE: track 0.00 -> 4.28 mm
- net A+: track 0.00 -> 3.36 mm
- net PG: track 0.00 -> 3.29 mm
- net A-: track 0.00 -> 3.24 mm
- net Net-(U2-PA15): track 0.00 -> 3.03 mm
- net USART1_TX: track 0.00 -> 2.24 mm
- net USART1_RX: track 0.00 -> 2.01 mm
- net Net-(U2-PF0): track 0.00 -> 1.88 mm
- net Net-(D2-A): track 0.00 -> 1.68 mm
- net Net-(D1-A): track 0.00 -> 1.67 mm

Commit message: lqwkrjfsadklj
Parts:
- moved C9 63.1 mm to (181.4, 60.0), turned to 90 degrees
- moved C8 56.9 mm to (175.3, 59.6), turned to 90 degrees
- moved C7 53.4 mm to (172.8, 59.6), turned to 90 degrees
- moved C6 49.9 mm to (170.3, 59.6), turned to 90 degrees
- moved C5 46.4 mm to (167.8, 59.6), turned to 90 degrees
- moved C4 43.0 mm to (165.2, 59.6), turned to 90 degrees
- moved C10 11.2 mm to (179.9, 88.4)
- moved C11 11.2 mm to (179.9, 90.0)
- moved R10 0.92 mm to (180.0, 92.3)
- moved R7 0.92 mm to (168.0, 94.1)
- moved R8 0.92 mm to (168.1, 95.5)
- moved R5 0.92 mm to (168.1, 91.0)
- moved R6 0.92 mm to (168.1, 92.6)
- moved R9 0.92 mm to (180.0, 93.8)
- moved U3 0.92 mm to (173.5, 93.1)
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
Commit message: goodie
going good
Parts:
- moved C9 27.5 mm to (164.5, 81.7), turned to 0 degrees
- moved C8 23.3 mm to (164.5, 80.2), turned to 0 degrees
- moved C5 20.2 mm to (155.4, 75.6), turned to -90 degrees
- moved C7 12.0 mm to (169.5, 71.1)
- moved C6 11.8 mm to (168.0, 71.1)
- moved C4 9.32 mm to (159.7, 67.1), turned to 180 degrees
- moved U4 1.78 mm to (152.8, 74.1)
- moved C1 1.70 mm to (152.8, 76.4)
Routing:
- net USART1_TX: track 2.24 -> 61.6 mm, vias 0 -> 2
- net SWDIO: track 0.00 -> 29.4 mm, vias 0 -> 2
- net ALERT1: track 0.00 -> 28.7 mm, vias 0 -> 2
- net SWCLK: track 0.00 -> 27.4 mm, vias 0 -> 2
- net A-: track 3.24 -> 29.8 mm
- net NRST_PSB: track 0.00 -> 25.4 mm, vias 0 -> 1
- net I2C1_SDA: track 0.00 -> 24.3 mm
- net A+: track 3.36 -> 24.0 mm
- net PG: track 3.29 -> 20.7 mm
- net I2C1_SCL: track 0.00 -> 15.2 mm
- net 3.3V: track 10.0 -> 23.6 mm
- net GND: track 5.40 -> 18.0 mm
- net Net-(U2-PF0): track 1.88 -> 3.66 mm

Commit message: finished!!!! RAHHHH
RAHHHHHHHHHHH
Parts:
- moved C10 2.00 mm to (178.2, 87.4)
- moved R5 2.00 mm to (166.4, 90.0)
- moved R6 2.00 mm to (166.3, 91.6)
- moved R9 2.00 mm to (178.2, 92.8)
- moved R10 2.00 mm to (178.3, 91.3)
- moved R11 2.00 mm to (176.0, 92.1)
- moved R8 2.00 mm to (166.4, 94.5)
- moved U3 2.00 mm to (171.7, 92.1)
- moved C11 2.00 mm to (178.2, 89.0)
- moved R7 2.00 mm to (166.3, 93.0)
- moved D1 0.15 mm to (168.3, 67.3)
Routing:
- net 5V: track 5.57 -> 81.7 mm, vias 1 -> 7
- net GND: track 18.0 -> 89.3 mm, vias 1 -> 14
- net 3.3V: track 23.6 -> 72.6 mm, vias 0 -> 21
- net USART1_RX: track 2.01 -> 38.3 mm, vias 0 -> 2
- net USART1_DE: track 4.28 -> 38.8 mm, vias 0 -> 2
- net SWDIO: track 29.4 -> 62.7 mm, vias 2 -> 5
- net NRST_PSB: track 25.4 -> 52.3 mm, vias 1 -> 2
- net SWCLK: track 27.4 -> 50.7 mm, vias 2 -> 3
- net A-: track 29.8 -> 23.4 mm, vias 0 -> 2
- net USART1_TX: track 61.6 -> 60.0 mm
- net I2C1_SCL: track 15.2 -> 16.4 mm, vias 0 -> 1
- net A+: track 24.0 -> 24.7 mm, vias 0 -> 1
- added copper zone on B.Cu, net 3.3V
- added copper zone on F.Cu, net 5V

Commit message: errors
no errors
Parts:
- moved R10 0.49 mm to (178.7, 91.2)
- moved R9 0.46 mm to (178.7, 92.8)
- moved R11 0.32 mm to (176.3, 92.0)
Routing:
- net A+: track 24.7 -> 25.3 mm
Changed lines of the file:
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@@
 		)
 		(property "Value" "0.1uF"
-			(at -2.2 0.27 360)
+			(at -2.2 0.27 0)
 			(layer "F.Fab")
 			(effects
@@
 		)
 		(fp_text user "${REFERENCE}"
-			(at 0 0 360)
+			(at 0 0 0)
 			(layer "F.Fab")
 			(effects
@@
 	(footprint "Resistor_SMD:R_0603_1608Metric_Pad0.98x0.95mm_HandSolder"
 		(layer "F.Cu")
-		(at 178.252 91.308264)
+		(at 178.73 91.22)
 		(descr "Resistor SMD 0603 (1608 Metric), square (rectangular) end terminal, IPC_7351 nominal with elongated pad for handsoldering. (Body size source: IPC-SM-782 page 72, https://www.pcb-3d.com/wordpress/wp-content/uploads/ipc-sm-782a_amendment_1_and_2.pdf), generated with kicad-footprint-generator")
 		(tags "resistor handsolder")
@@
 	(footprint "Resistor_SMD:R_0603_1608Metric_Pad0.98x0.95mm_HandSolder"
 		(layer "F.Cu")
-		(at 175.967 92.128264 -90)
+		(at 176.27 92.04 -90)
 		(descr "Resistor SMD 0603 (1608 Metric), square (rectangular) end terminal, IPC_7351 nominal with elongated pad for handsoldering. (Body size source: IPC-SM-782 page 72, https://www.pcb-3d.com/wordpress/wp-content/uploads/ipc-sm-782a_amendment_1_and_2.pdf), generated with kicad-footprint-generator")
 		(tags "resistor handsolder")
@@
 	(footprint "Resistor_SMD:R_0603_1608Metric_Pad0.98x0.95mm_HandSolder"
 		(layer "F.Cu")
-		(at 178.2445 92.778264 180)
+		(at 178.7 92.79 180)
 		(descr "Resistor SMD 0603 (1608 Metric), square (rectangular) end terminal, IPC_7351 nominal with elongated pad for handsoldering. (Body size source: IPC-SM-782 page 72, https://www.pcb-3d.com/wordpress/wp-content/uploads/ipc-sm-782a_amendment_1_and_2.pdf), generated with kicad-footprint-generator")
 		(tags "resistor handsolder")
@@
 		(tags "capacitor handsolder")
 		(property "Reference" "C8"
-			(at -1.7575 -0.23 360)
+			(at -1.7575 -0.23 0)
 			(layer "F.SilkS")
 			(effects
@@
 		)
 		(property "Value" "4.7uF"
-			(at -2.1675 0.23 360)
+			(at -2.1675 0.23 0)
 			(layer "F.Fab")
 			(effects
@@
 		)
 		(fp_text user "${REFERENCE}"
-			(at 0 0 360)
+			(at 0 0 0)
 			(layer "F.Fab")
 			(effects
@@
 		(tags "capacitor handsolder")
 		(property "Reference" "C4"
-			(at 1.74 0.25 360)
+			(at 1.74 0.25 0)
 			(layer "F.SilkS")
 			(effects
@@
 		)
 		(property "Value" "0.1uF"
-			(at 2.16 -0.24 360)
+			(at 2.16 -0.24 0)
 			(layer "F.Fab")
 			(effects
@@
 		)
 		(fp_text user "${REFERENCE}"
-			(at 0 0 360)
+			(at 0 0 0)
 			(layer "F.Fab")
 			(effects
@@
 	)
 	(segment
-		(start 178.398 86.358514)
-		(end 179.712616 86.358514)
+		(start 175.867 89.870682)
+		(end 174.499582 89.870682)
 		(width 0.762)
 		(layer "F.Cu")
@@
 	)
 	(segment
-		(start 175.867 90.138264)
-		(end 175.867 89.870682)
+		(start 178.398 86.358514)
+		(end 179.712616 86.358514)
 		(width 0.762)
 		(layer "F.Cu")
@@
 	)
 	(segment
-		(start 175.24 89.243682)
-		(end 175.24 88.46)
+		(start 180.2725 67.84)
+		(end 176.65 67.84)
 		(width 0.762)
 		(layer "F.Cu")
@@
 	)
 	(segment
-		(start 180.2725 67.84)
-		(end 176.65 67.84)
+		(start 163.31 93.08)
+		(end 165.367764 93.08)
 		(width 0.762)
 		(layer "F.Cu")
@@
 	)
 	(segment
-		(start 163.31 93.08)
-		(end 165.367764 93.08)
+		(start 165.4795 89.978264)
+		(end 163.257 89.978264)
 		(width 0.762)
 		(layer "F.Cu")
@@
 	)
 	(segment
-		(start 174.232 90.138264)
-		(end 175.867 90.138264)
+		(start 178.33 86.426514)
+		(end 177.342 87.414514)
 		(width 0.762)
 		(layer "F.Cu")
@@
 	)
 	(segment
-		(start 165.4795 89.978264)
-		(end 163.257 89.978264)
+		(start 174.499582 89.870682)
+		(end 174.222 90.148264)
 		(width 0.762)
 		(layer "F.Cu")
@@
 	)
 	(segment
-		(start 178.33 86.426514)
-		(end 177.342 87.414514)
+		(start 175.24 89.243682)
+		(end 175.24 88.46)
 		(width 0.762)
 		(layer "F.Cu")
@@
 	)
 	(segment
-		(start 174.222 90.148264)
-		(end 174.232 90.138264)
-		(width 0.762)
-		(layer "F.Cu")
-		(net 7)
-	)
-	(segment
 		(start 175.867 89.870682)
 		(end 175.24 89.243682)
@@
 	)
 	(via
-		(at 175.867 90.138264)
+		(at 175.867 89.870682)
 		(size 0.6)
 		(drill 0.3)
@@
 	)
 	(segment
-		(start 175.867 90.138264)
-		(end 175.867 88.753)
-		(width 0.762)
-		(layer "B.Cu")
-		(net 7)
-	)
-	(segment
 		(start 161.285264 92.475264)
 		(end 163.29 94.48)
@@
 	)
 	(segment
+		(start 175.867 89.870682)
+		(end 175.867 88.753)
+		(width 0.762)
+		(layer "B.Cu")
+		(net 7)
+	)
+	(segment
 		(start 161.285264 91.96)
 		(end 162.307 90.938264)
@@
 	)
 	(segment
-		(start 178.207 91.903264)
-		(end 177.332 92.778264)
+		(start 177.784014 89.784014)
+		(end 178.7 90.7)
 		(width 0.254)
 		(layer "F.Cu")
@@
 	)
 	(segment
-		(start 177.303654 89.784014)
-		(end 178.207 90.68736)
+		(start 175.6145 92.688264)
+		(end 175.967 93.040764)
 		(width 0.254)
 		(layer "F.Cu")
@@
 	)
 	(segment
-		(start 175.6145 92.688264)
-		(end 175.967 93.040764)
+		(start 178.7 90.7)
+		(end 178.7 92.01)
 		(width 0.254)
 		(layer "F.Cu")
@@
 	)
 	(segment
-		(start 177.449 76.65)
-		(end 177.449 78.2835)
+		(start 176.781596 89.784014)
+		(end 177.784014 89.784014)
 		(width 0.254)
 		(layer "F.Cu")
@@
 	)
 	(segment
-		(start 176.781596 89.784014)
-		(end 177.303654 89.784014)
+		(start 177.449 76.65)
+		(end 177.449 78.2835)
 		(width 0.254)
 		(layer "F.Cu")
@@
 	)
 	(segment
-		(start 176.4575 89.459918)
-		(end 176.781596 89.784014)
+		(start 177.92 92.79)
+		(end 177.7875 92.79)
 		(width 0.254)
 		(layer "F.Cu")
@@
 	)
 	(segment
-		(start 177.21 78.5225)
-		(end 177.21 85.70011)
+		(start 177.449 78.2835)
+		(end 177.21 78.5225)
 		(width 0.254)
 		(layer "F.Cu")
@@
 	)
 	(segment
-		(start 177.449 78.2835)
-		(end 177.21 78.5225)
+		(start 177.21 85.70011)
+		(end 176.4575 86.45261)
 		(width 0.254)
 		(layer "F.Cu")
@@
 	)
 	(segment
-		(start 177.21 85.70011)
-		(end 176.4575 86.45261)
+		(start 174.222 92.688264)
+		(end 175.6145 92.688264)
 		(width 0.254)
 		(layer "F.Cu")
@@
 	)
 	(segment
-		(start 174.222 92.688264)
-		(end 175.6145 92.688264)
+		(start 177.21 78.5225)
+		(end 177.21 85.70011)
 		(width 0.254)
 		(layer "F.Cu")
@@
 	)
 	(segment
-		(start 178.207 90.68736)
-		(end 178.207 91.903264)
+		(start 178.7 92.01)
+		(end 177.92 92.79)
+		(width 0.254)
+		(layer "F.Cu")
+		(net 11)
+	)
+	(segment
+		(start 176.4575 89.459918)
+		(end 176.781596 89.784014)
 		(width 0.254)
 		(layer "F.Cu")
@@
 	)
 	(segment
-		(start 179.1645 91.308264)
-		(end 179.1645 89.099514)
-		(width 0.762)
-		(layer "F.Cu")
-		(net 40)
-	)
-	(segment
 		(start 158.25 74.94)
 		(end 159.07 75.76)
@@
 	)
 	(segment
+		(start 179.1645 89.099514)
+		(end 179.047 88.982014)
+		(width 0.762)
+		(layer "F.Cu")
+		(net 40)
+	)
+	(segment
 		(start 160.053592 68.963)
 		(end 160.31 69.219408)
@@
 	)
 	(segment
-		(start 179.1645 89.099514)
-		(end 179.047 88.982014)
-		(width 0.762)
-		(layer "F.Cu")
-		(net 40)
-	)
-	(segment
 		(start 163.6175 80.18)
 		(end 161.07 80.18)
@@
 	)
 	(segment
-		(start 179.1645 91.308264)
-		(end 180.168264 91.308264)
+		(start 180.315 89.865)
+		(end 179.549514 89.099514)
 		(width 0.762)
 		(layer "F.Cu")
@@
 	)
 	(segment
-		(start 180.18 91.32)
-		(end 180.168264 91.308264)
-		(width 0.762)
-		(layer "F.Cu")
-		(net 40)
-	)
-	(segment
 		(start 160.63 70.0275)
 		(end 160.63 71.09)
@@
 	)
 	(segment
+		(start 180.315 91.185)
+		(end 180.18 91.32)
+		(width 0.762)
+		(layer "F.Cu")
+		(net 40)
+	)
+	(segment
 		(start 163.81 79.9875)
 		(end 163.6175 80.18)
@@
 	)
 	(segment
+		(start 180.315 89.865)
+		(end 180.315 91.185)
+		(width 0.762)
+		(layer "F.Cu")
+		(net 40)
+	)
+	(segment
+		(start 179.549514 89.099514)
+		(end 179.1645 89.099514)
+		(width 0.762)
+		(layer "F.Cu")
+		(net 40)
+	)
+	(segment
 		(start 159.31 70.0275)
 		(end 159.31 69.219408)
@@
 	)
 	(via
-		(at 180.168264 91.308264)
+		(at 180.315 89.865)
 		(size 0.6)
 		(drill 0.3)

Commit message: Update X17-Data-Conversion.kicad_pcb
uipdate
Routing:
- net GND: track 89.1 -> 80.8 mm, vias 14 -> 15
Changed lines of the file:
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@@
+	)
+	(segment
+		(start 142.8475 67.84)
+		(end 143.28 67.84)
+		(width 0.762)
+		(layer "F.Cu")
+		(net 40)
 	)
 	(segment
@@
 	)
 	(segment
+		(start 143.28 67.84)
+		(end 143.31 67.81)
+		(width 0.762)
+		(layer "F.Cu")
+		(net 40)
+	)
+	(segment
 		(start 150.86 75.75)
 		(end 151.819 76.709)
@@
 	)
 	(via
+		(at 145.01 68.5)
+		(size 0.6)
+		(drill 0.3)
+		(layers "F.Cu" "B.Cu")
+		(net 40)
+	)
+	(via
 		(at 160.61 71.11)
 		(size 0.6)
@@
 	(segment
 		(start 142.8475 67.84)
+		(end 144.35 67.84)
+		(width 0.762)
+		(layer "B.Cu")
+		(net 40)
+	)
+	(segment
+		(start 142.8475 67.84)
 		(end 142.95 67.84)
 		(width 0.762)
@@
 	)
 	(segment
-		(start 142.95 67.84)
-		(end 150.86 75.75)
-		(width 0.762)
-		(layer "B.Cu")
+		(start 144.35 67.84)
+		(end 145.01 68.5)
+		(width 0.762)
+		(layer "B.Cu")

Commit message: daniel lookie
Connections:
- J4 pad 10: A+ -> NRST_PSB
- J4 pad 11: A- -> A+
- J4 pad 12: NRST_PSB -> A-
- J4 pad 3: SWDIO -> unconnected-(J4-Pin_3-Pad3)
- J4 pad 4: SWCLK -> unconnected-(J4-Pin_4-Pad4)
Routing:
- net A-: track 23.4 -> 18.7 mm, vias 2 -> 1
- net A+: track 25.3 -> 22.8 mm
- net NRST_PSB: track 52.3 -> 51.3 mm
Changed lines of the file:
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@@
 	(net 44 "Net-(U2-PF0)")
 	(net 45 "unconnected-(U2-PF1-Pad6)")
+	(net 46 "unconnected-(J4-Pin_3-Pad3)")
+	(net 47 "unconnected-(J4-Pin_4-Pad4)")
 	(footprint "Capacitor_SMD:C_0603_1608Metric_Pad1.08x0.95mm_HandSolder"
 		(layer "F.Cu")
@@
 			(layers "*.Cu" "*.Mask")
 			(remove_unused_layers no)
-			(net 5 "SWDIO")
+			(net 46 "unconnected-(J4-Pin_3-Pad3)")
 			(pinfunction "Pin_3")
-			(pintype "passive")
+			(pintype "passive+no_connect")
 		)
 		(pad "4" thru_hole oval
@@
 			(layers "*.Cu" "*.Mask")
 			(remove_unused_layers no)
-			(net 4 "SWCLK")
+			(net 47 "unconnected-(J4-Pin_4-Pad4)")
 			(pinfunction "Pin_4")
-			(pintype "passive")
+			(pintype "passive+no_connect")
 		)
 		(pad "5" thru_hole oval
@@
 			(layers "*.Cu" "*.Mask")
 			(remove_unused_layers no)
-			(net 11 "A+")
+			(net 1 "NRST_PSB")
 			(pinfunction "Pin_10")
 			(pintype "passive")
@@
 			(layers "*.Cu" "*.Mask")
 			(remove_unused_layers no)
-			(net 12 "A-")
+			(net 11 "A+")
 			(pinfunction "Pin_11")
 			(pintype "passive")
@@
 			(layers "*.Cu" "*.Mask")
 			(remove_unused_layers no)
-			(net 1 "NRST_PSB")
+			(net 12 "A-")
 			(pinfunction "Pin_12")
 			(pintype "passive")
@@
 		)
 		(property "Value" "MAX7375AXR805+T"
-			(at 1.21 -2.07 90)
+			(at 0 0 90)
 			(unlocked yes)
 			(layer "F.Fab")
 			(effects
 				(font
-					(size 0.381 0.381)
-					(thickness 0.03175)
+					(size 1 1)
+					(thickness 0.15)
 				)
 			)
@@
 	)
 	(segment
-		(start 159.483 75.03)
-		(end 174.7625 75.03)
+		(start 177.449 76.65)
+		(end 177.46 76.65)
+		(width 0.254)
+		(layer "B.Cu")
+		(net 1)
+	)
+	(segment
+		(start 177.46 76.65)
+		(end 177.570224 76.760224)
+		(width 0.254)
+		(layer "B.Cu")
+		(net 1)
+	)
+	(segment
+		(start 177.570224 76.760224)
+		(end 178.972276 76.760224)
 		(width 0.254)
 		(layer "B.Cu")
@@
 	(segment
 		(start 159.483 75.03)
-		(end 159.473 75.04)
+		(end 175.829 75.03)
 		(width 0.254)
 		(layer "B.Cu")
@@
 	)
 	(segment
-		(start 174.7625 75.03)
-		(end 180.2725 80.54)
+		(start 175.829 75.03)
+		(end 177.449 76.65)
+		(width 0.254)
+		(layer "B.Cu")
+		(net 1)
+	)
+	(segment
+		(start 178.972276 76.760224)
+		(end 180.2725 75.46)
+		(width 0.254)
+		(layer "B.Cu")
+		(net 1)
+	)
+	(segment
+		(start 159.483 75.03)
+		(end 159.473 75.04)
 		(width 0.254)
 		(layer "B.Cu")
@@
 	)
 	(segment
-		(start 177.784014 89.784014)
-		(end 178.7 90.7)
-		(width 0.254)
-		(layer "F.Cu")
-		(net 11)
-	)
-	(segment
 		(start 175.6145 92.688264)
 		(end 175.967 93.040764)
@@
 	)
 	(segment
-		(start 178.7 90.7)
-		(end 178.7 92.01)
-		(width 0.254)
-		(layer "F.Cu")
-		(net 11)
-	)
-	(segment
-		(start 176.781596 89.784014)
-		(end 177.784014 89.784014)
+		(start 173.247001 92.688264)
+		(end 174.222 92.688264)
 		(width 0.254)
 		(layer "F.Cu")
@@
 	)
 	(segment
-		(start 177.449 76.65)
-		(end 177.449 78.2835)
+		(start 177.25 80.92)
+		(end 172.466 85.704)
 		(width 0.254)
 		(layer "F.Cu")
@@
 	)
 	(segment
-		(start 177.449 78.2835)
-		(end 177.21 78.5225)
-		(width 0.254)
-		(layer "F.Cu")
-		(net 11)
-	)
-	(segment
-		(start 176.4575 86.45261)
-		(end 176.4575 89.459918)
+		(start 172.466 91.907263)
+		(end 173.247001 92.688264)
 		(width 0.254)
 		(layer "F.Cu")
@@
 	)
 	(segment
-		(start 177.21 85.70011)
-		(end 176.4575 86.45261)
+		(start 177.27 80.92)
+		(end 177.25 80.92)
 		(width 0.254)
 		(layer "F.Cu")
@@
 	)
 	(segment
-		(start 177.21 78.5225)
-		(end 177.21 85.70011)
-		(width 0.254)
-		(layer "F.Cu")
-		(net 11)
-	)
-	(segment
-		(start 178.7 92.01)
-		(end 177.92 92.79)
-		(width 0.254)
-		(layer "F.Cu")
-		(net 11)
-	)
-	(segment
-		(start 176.4575 89.459918)
-		(end 176.781596 89.784014)
+		(start 172.466 85.704)
+		(end 172.466 91.907263)
 		(width 0.254)
 		(layer "F.Cu")
@@
 	)
 	(via
-		(at 177.449 76.65)
+		(at 177.27 80.92)
 		(size 0.6)
 		(drill 0.3)
@@
 	)
 	(segment
-		(start 178.972276 76.760224)
-		(end 177.570224 76.760224)
-		(width 0.254)
-		(layer "B.Cu")
-		(net 11)
-	)
-	(segment
-		(start 177.46 76.65)
-		(end 177.449 76.65)
-		(width 0.254)
-		(layer "B.Cu")
-		(net 11)
-	)
-	(segment
-		(start 180.2725 75.46)
-		(end 178.972276 76.760224)
+		(start 177.3525 80.92)
+		(end 180.2725 78)
 		(width 0.254)
 		(layer "B.Cu")
@@
 	)
 	(segment
-		(start 177.570224 76.760224)
-		(end 177.46 76.65)
+		(start 177.27 80.92)
+		(end 177.3525 80.92)
 		(width 0.254)
 		(layer "B.Cu")
@@
 	)
 	(segment
-		(start 175.163 85.54)
-		(end 174.643 86.06)
-		(width 0.254)
-		(layer "F.Cu")
-		(net 12)
-	)
-	(segment
-		(start 174.643 86.06)
-		(end 172.92 87.783)
+		(start 173.247001 91.418264)
+		(end 174.222 91.418264)
 		(width 0.254)
 		(layer "F.Cu")
@@
 	)
 	(segment
-		(start 175.29 85.54)
-		(end 175.163 85.54)
+		(start 172.92 87.783)
+		(end 172.92 91.091263)
 		(width 0.254)
 		(layer "F.Cu")
@@
 	)
 	(segment
-		(start 181.4495 79.177)
-		(end 181.4495 81.2805)
-		(width 0.254)
-		(layer "F.Cu")
-		(net 12)
-	)
-	(segment
 		(start 175.967 91.215764)
 		(end 177.247 91.215764)
@@
 	)
 	(segment
-		(start 180.2725 78)
-		(end 181.4495 79.177)
+		(start 177.253 83.45)
+		(end 172.92 87.783)
 		(width 0.254)
 		(layer "F.Cu")
@@
 	)
 	(segment
-		(start 173.247001 91.418264)
-		(end 174.222 91.418264)
+		(start 177.38 83.45)
+		(end 177.253 83.45)
 		(width 0.254)
 		(layer "F.Cu")
@@
 	)
 	(segment
-		(start 181.4495 81.2805)
-		(end 179.68 83.05)
-		(width 0.254)
-		(layer "F.Cu")
-		(net 12)
-	)
-	(segment
-		(start 172.92 87.783)
-		(end 172.92 91.091263)
-		(width 0.254)
-		(layer "F.Cu")
-		(net 12)
-	)
-	(segment
 		(start 173.838264 91.418264)
 		(end 174.222 91.418264)
@@
 	)
 	(via
-		(at 179.68 83.05)
-		(size 0.6)
-		(drill 0.3)
-		(layers "F.Cu" "B.Cu")
-		(net 12)
-	)
-	(via
-		(at 175.29 85.54)
+		(at 177.38 83.45)
 		(size 0.6)
 		(drill 0.3)
@@
 	)
 	(segment
-		(start 179.68 83.05)
-		(end 177.78 83.05)
+		(start 180.2725 80.5575)
+		(end 180.2725 80.54)
 		(width 0.254)
 		(layer "B.Cu")
@@
 	)
 	(segment
-		(start 177.78 83.05)
-		(end 175.29 85.54)
+		(start 177.38 83.45)
+		(end 180.2725 80.5575)
 		(width 0.254)
 		(layer "B.Cu")
