File: X17-Data-Conversion.kicad_pcb (KiCad board)
At the start: 2 copper layers, 41.5 x 30.7 mm, 28 parts, among them J1 Conn_01x05, J4 Conn_01x12_Pin, U2 STM32F091CCTx, U3 MAX485E, U4 MAX7375AXR805+T, U5 AZ1117IH-3.3TRG1

Commit message: 1/10/25 gerber files
Routing:
- net SWCLK: track 50.7 -> 45.8 mm, vias 3 -> 4
- net SWDIO: track 62.7 -> 64.9 mm, vias 5 -> 6
- net NRST_PSB: track 51.3 -> 53.3 mm
- net 5V: track 81.2 -> 79.6 mm
- net GND: track 80.8 -> 79.6 mm
- net I2C1_SDA: track 24.3 -> 25.2 mm
- net ALERT1: track 28.7 -> 29.3 mm
